File: mk_01/v0.1/Hardware/mk_01_LHS/mk_01_LHS.kicad_sch (KiCad schematic)
At the start: 98 parts, among them IC1 DIO6605BFN8, Q1 2N7000, SW1 SW_Push_Dual, U1 nice_nano

Commit message: Updates
Incldues updates to ZMK and the creation of the BlueMicro firmware folder
Other:
- company: (none) -> Bangor University
- title: (none) -> mk_01_LHS
Changed lines of the file:
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@@
 (kicad_sch (version 20211123) (generator eeschema)
   (paper "A3")
+  (title_block
+    (title "mk_01_LHS")
+    (date "2022-05-12")
+    (rev "v0.1")
+    (company "Bangor University")
+  )
   (junction (at 205.74 198.12) (diameter 0) (color 0 0 0 0)
   )
